Commit message: Moved get_tag_distance to directory to enable launching with ros2 run, added tag_test_monitor.py as well as calibration file for simple camera at home + map for home test area.  Additionally included script to generate maps and tag maps.

File: 2026/code/ros_package/team9214_ws/src/arena_description/urdf/robot.urdf.lab.test.xacro (robot description, xacro)
@@ -4,5 +4,7 @@
   <!--
     Test setup
-      Camera: 36inches from the floor, so 0.8636 m
+      Camera: 90cm from floor
+      AprilTag: 110cm from floor
+      AprilTag: 150cm in front of camera
   -->
   <!-- Camera 1 (forward) -->
@@ -13,5 +15,5 @@
     <!-- Replace with your measured/calibrated extrinsics -->
     <!-- +x forward, +y left, +z up -->
-    <origin xyz="0.00 0.00 0.8636" rpy="0 0 0"/>
+    <origin xyz="0.00 0.00 0.90" rpy="0 0 0"/>
   </joint>
   <link name="camera_1_optical_frame"/>
